Commit message: car car car

File: resources/car.urdf (robot description, URDF)
Before this commit: robot car, 7 links, 6 joints
Links:
- link base_link: geometry visual box size=0.08 0.4 0.01; visual box size=0.08 0.45 0.01
- link left_back_wheel: geometry collision cylinder length=0.05 radius=0.1; visual cylinder length=0.08 radius=0.11
- link left_front_wheel: geometry collision cylinder length=0.05 radius=0.1; visual cylinder length=0.06 radius=0.09
- link right_back_wheel: geometry collision cylinder length=0.05 radius=0.1; visual cylinder length=0.08 radius=0.11
- link right_front_wheel: geometry collision cylinder length=0.05 radius=0.1; visual cylinder length=0.06 radius=0.09
